File: PCBFiles+Schematics/Main PCB/info_orbs.kicad_sch (KiCad schematic)
At the start: 13 parts, among them J1 Conn_01x02_Pin, SW1 SW_Push, SW2 SW_Push, SW3 SW_Push

Commit message: Reopen the S3 variant at Yang's request; repo renamed to hot-info-orbs
The decline was made on cost and complexity, not a technical blocker, and the
objection that carried the most weight now looks answerable for free. The
GC9A01 clone modules appear to carry their own onboard regulator, so the
displays can run from a 5V bus off the module's 5V pin and drop to 3.3V
individually -- spreading ~0.1W across five packages instead of concentrating
~0.5W in the SuperMini's LDO, which then carries only the ESP32. No added
regulator, no carrier-board complexity, which is exactly the budget that closed
this the first time.

Records what must be measured rather than assumed, because "GC9A01 clone from
AliExpress" is not a specification: inventory already holds one generic module
recorded as 3.3V-only and another as 3.3/5V with an 8-pin BL interface. Same
controller, different power design.

Proposed pin map moves the bus off IO1-10 so all six spare ADC1 pins stay
available, and keeps the buttons off IO3, which HackerBoxes used despite it
being an S3 strapping pin.

Earlier decision record kept rather than deleted -- the reasoning that reversed
is the useful part.
Parts:
- U1, USBPower1, tft1, tft2, tft3, tft4, tft5: value ~ -> (none)
