File: hardware/hot-info-orbs/hot_info_orbs.kicad_sch (KiCad schematic)
At the start: 10 parts, among them SW1 SW_Push, SW2 SW_Push, SW3 SW_Push, U2 ESP32-S3-SuperMini

Commit message: Board fixes: DS5 DC connected, button off the strapping pin, GND pour added
Three changes to Yang's Rev 1.0, all verified against the file and by re-running
KiCad's own checks -- ERC 0, DRC 0, 0 unconnected pads, 0 schematic parity
issues, and the three silkscreen warnings cleared too.

DS5 pin 5 (DC) now lands on Net-(DS1-DC). The wire had been drawn but stopped
3.81mm short of the pin, so the fifth display had no data/command line. Worth
noting DRC could never have caught it: the board faithfully implemented the
schematic, and the gap was in the schematic. Only ERC sees that class.

SW3 moved from GPIO3 to GPIO10. GPIO3 is an ESP32-S3 strapping pin and the
buttons pull high, so holding that button during a reset drove a strapping pin
at boot -- the shape of an intermittent no-boot nobody traces to a button.
GPIO10 was already broken out and unused.

GND pour on B.Cu, and a SECOND antenna keepout added on B.Cu. The original
keepout was F.Cu only and set to copperpour allowed, so a back-side pour would
have filled straight under the SuperMini's antenna -- the one thing the keepout
exists to prevent. Both layers now exclude copper fill.

Vias went 20 -> 21 rather than down, because the original GND traces remain
alongside the pour. Deliberately not rerouting: via count only mattered while
milling was under consideration, and this board is going to JLCPCB where vias
are free. Wholesale rerouting someone else's board is also far harder to review
than three targeted fixes.
Connections:
- net at DS5.5 (DC): now also DS1.5 (DC), DS2.5 (DC), DS3.5 (DC), DS4.5 (DC), U2.8 (GPIO_9)
- net at U2.14 (GPIO_3): no longer SW3.1
- net SW3: now reaches U2.7 (GPIO_10)
- net SW3: now also SW3.1
- no-connect marks 0 -> 3
Changed lines of the file:
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@@
+	)
+	(junction
+		(at 175.26 53.34)
+		(diameter 0)
+		(color 0 0 0 0)
+	)
+	(junction
+		(at 177.8 55.88)
+		(diameter 0)
+		(color 0 0 0 0)
 	)
 	(junction
@@
 	)
 	(junction
-		(at 175.26 53.34)
-		(diameter 0)
-		(color 0 0 0 0)
-	)
-	(junction
-		(at 177.8 55.88)
-		(diameter 0)
-		(color 0 0 0 0)
-	)
-	(junction
 		(at 92.71 132.08)
 		(diameter 0)
@@
 		(color 0 0 0 0)
 	)
+	(no_connect
+		(at 96.52 80.01)
+	)
+	(no_connect
+		(at 96.52 83.82)
+	)
+	(no_connect
+		(at 96.52 95.25)
+	)
 	(wire
 		(pts
@@
 	(wire
 		(pts
-			(xy 172.72 43.18) (xy 172.72 50.8)
-		)
-		(stroke
-			(width 0)
-			(type default)
-		)
-	)
-	(wire
-		(pts
 			(xy 118.11 55.88) (xy 118.11 46.99)
 		)
@@
 	(wire
 		(pts
-			(xy 49.53 95.25) (xy 96.52 95.25)
-		)
-		(stroke
-			(width 0)
-			(type default)
-		)
-	)
-	(wire
-		(pts
 			(xy 93.98 60.96) (xy 123.19 60.96)
 		)
@@
 	(wire
 		(pts
+			(xy 127 102.87) (xy 134.62 102.87)
+		)
+		(stroke
+			(width 0)
+			(type default)
+		)
+	)
+	(wire
+		(pts
 			(xy 81.28 102.87) (xy 96.52 102.87)
 		)
@@
 	(wire
 		(pts
-			(xy 74.93 157.48) (xy 49.53 157.48)
-		)
-		(stroke
-			(width 0)
-			(type default)
-		)
-	)
-	(wire
-		(pts
 			(xy 63.5 58.42) (xy 63.5 46.99)
 		)
@@
 	(wire
 		(pts
+			(xy 66.04 157.48) (xy 74.93 157.48)
+		)
+		(stroke
+			(width 0)
+			(type default)
+		)
+	)
+	(wire
+		(pts
 			(xy 137.16 48.26) (xy 107.95 48.26)
 		)
@@
 	(wire
 		(pts
-			(xy 49.53 95.25) (xy 49.53 157.48)
-		)
-		(stroke
-			(width 0)
-			(type default)
-		)
-	)
-	(wire
-		(pts
 			(xy 196.85 83.82) (xy 203.2 83.82)
 		)
@@
 	(wire
 		(pts
+			(xy 172.72 46.99) (xy 172.72 50.8)
+		)
+		(stroke
+			(width 0)
+			(type default)
+		)
+	)
+	(wire
+		(pts
 			(xy 92.71 127) (xy 160.02 127)
 		)
@@
 		)
 	)
+	(label "SW3"
+		(at 134.62 102.87 0)
+		(effects
+			(font
+				(size 1.27 1.27)
+			)
+			(justify left bottom)
+		)
+	)
+	(label "SW3"
+		(at 66.04 157.48 0)
+		(effects
+			(font
+				(size 1.27 1.27)
+			)
+			(justify left bottom)
+		)
+	)

Commit message: Yang's v2: near-complete reroute, DS5 fixed, real logo library, 3D models
Second board from Yang, received while we were fixing the first. He reworked
the routing substantially -- 192 of 211 track segments removed and 197 added,
against 19 segments in common with our version -- and moved signal copper onto
F.Cu, dropping B.Cu from 309mm to 221mm. That leaves the back layer clearer
than v1 did, which suits the ground pour better than his original would have.

He fixed DS5's DC pin independently. He did not move the button off GPIO3 and
did not add a pour, so those two of our three changes still need re-applying
on top of this; that is the next commit rather than this one, so his work and
ours stay separable in the history.

This commit takes his board wholesale rather than merging: KiCad files do not
merge, and reproducing his reroute would cost far more than re-applying two
well-understood edits.

Also brings the Hot_Logo_5x5mm library he had omitted from the first zip --
replacing the copy recovered out of the board cache -- plus STEP models for the
SuperMini and the display.

3D model paths rewritten from ${KICAD_USER_3DMODEL_DIR} to ${KIPRJMOD}/lib/3d.
His pointed at a directory on his own machine, the same portability problem the
symbol and footprint libraries had. Models do not affect fabrication, but a
project that renders for one person and not the other is the thing this layout
was set up to avoid.
Connections:
- net at U2.14 (GPIO_3): now also SW3.1
- net SW3: no longer names the net of U2.7 (GPIO_10)
- net SW3: no longer SW3.1
- no-connect marks 3 -> 0
Other:
- moved on the sheet: C1, DS1, DS2, DS3, DS4, DS5, SW1, SW2, SW3, U2

Commit message: v1.1 first production run: SW3 to GPIO10, pour filled, gerbers generated
Board is Yang's v1.1 with the three changes settled: SW3 moved off GPIO3, which
is an ESP32-S3 strapping pin the buttons would have driven high at reset;
GPIO3 now unconnected and GPIO10 carries the button. GND pour on B.Cu, filled.
Antenna keepout mirrored onto B.Cu and both layers set to block copper fill --
his original was F.Cu only and allowed the pour, which would have flooded copper
under the antenna the keepout exists to protect. Yang's leftover 3.81mm wire
stub from his own DS5 fix is gone.

Verified rather than assumed: ERC 0, DRC 0 unconnected pads, 0 schematic parity
issues. One silkscreen overlap on B.Silkscreen near U2 accepted as cosmetic.

Drill file cross-checks exactly against the footprints -- 18 vias at 0.30, 2 at
0.80 for C1, 53 at 1.00 for the display headers and module pins, 12 at 1.10 for
the buttons, 85 total. The four mounting holes are absent by design; they are
Edge.Cuts circles the fab routes.

The zip is named for the run and is not to be regenerated. If the board changes
the next run gets its own zip and tag, and this one stays byte-identical to what
was ordered -- so that when a board comes back there is no question what was
sent.

Carried knowingly into this run: 0.6/0.3 vias give a 0.150mm annular ring
against JLCPCB's stated 0.18mm. Recorded in fab/README as the first thing to
examine if these boards have via problems.
Connections:
- net at U2.14 (GPIO_3): no longer SW3.1
- net SW3: now reaches U2.7 (GPIO_10)
- net SW3: now also SW3.1
- no-connect marks 0 -> 3
Changed lines of the file:
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@@
-	)
-	(junction
-		(at 172.72 60.96)
-		(diameter 0)
-		(color 0 0 0 0)
 	)
 	(junction
@@
 		(color 0 0 0 0)
 	)
+	(no_connect
+		(at 96.52 109.22)
+	)
+	(no_connect
+		(at 96.52 93.98)
+	)
+	(no_connect
+		(at 96.52 97.79)
+	)
 	(wire
 		(pts
@@
 	(wire
 		(pts
-			(xy 172.72 57.15) (xy 172.72 60.96)
-		)
-		(stroke
-			(width 0)
-			(type default)
-		)
-	)
-	(wire
-		(pts
 			(xy 118.11 69.85) (xy 118.11 60.96)
 		)
@@
 	(wire
 		(pts
-			(xy 49.53 109.22) (xy 96.52 109.22)
-		)
-		(stroke
-			(width 0)
-			(type default)
-		)
-	)
-	(wire
-		(pts
 			(xy 93.98 74.93) (xy 123.19 74.93)
 		)
@@
 	(wire
 		(pts
-			(xy 74.93 171.45) (xy 49.53 171.45)
+			(xy 68.58 171.45) (xy 74.93 171.45)
 		)
 		(stroke
@@
 	(wire
 		(pts
-			(xy 49.53 109.22) (xy 49.53 171.45)
-		)
-		(stroke
-			(width 0)
-			(type default)
-		)
-	)
-	(wire
-		(pts
 			(xy 196.85 97.79) (xy 203.2 97.79)
 		)
@@
 		)
 	)
+	(wire
+		(pts
+			(xy 127 116.84) (xy 133.35 116.84)
+		)
+		(stroke
+			(width 0)
+			(type default)
+		)
+	)
+	(label "SW3"
+		(at 133.35 116.84 0)
+		(effects
+			(font
+				(size 1.27 1.27)
+			)
+			(justify left bottom)
+		)
+	)
+	(label "SW3"
+		(at 68.58 171.45 0)
+		(effects
+			(font
+				(size 1.27 1.27)
+			)
+			(justify left bottom)
+		)
+	)
