File: hardware/hot-info-orbs-xiao-46mm/hot_info_orbs_xiao_46mm.kicad_sch (KiCad schematic)
At the start: 12 parts, among them SW1 SW_Push, SW2 SW_Push, SW3 SW_Push, U2 XIAO ESP32-S3 Plus

Commit message: 46 mm board rev 2.5: probe pads for 3V3, GND and 5V
Scott wanted test pads for debugging other people's builds. RST, SCLK,
MOSI, DC and CS1-CS5 were suggested; his call: "just add gnd 3.3v and 5v".

TP1 3V3 / TP2 GND / TP3 5V sit in one column at x 173.74, between the
DS3 and DS4 display circles, at 2.54 mm pitch so a 1x3 header or clip
fits. GND is in the middle so the black probe stays put. Pads are 2.0 mm
on a 1.00 mm drill, the socket drill already on the board, so no new
tool (T4 49 -> 52). Rail names and a box are on both silks. With the
modules fitted the pads stay clear, but the front labels end up under
DS4. The back labels are always readable.

Rejected:
- the gap beside DS3 at x ~153: the pads clipped DS3's front silk circle;
- a 1x8 row with the bus signals: Scott's call.

Footprint lib/_TestPoints.pretty is the stock TestPoint THT pad trimmed
to stack at 2.54 mm: courtyard r 1.25, no silk circle, reference on
F.Fab. Rejected editing the stock footprint in the board: it leaves three
lib_footprint_mismatch warnings for good.

The schematic has a TEST POINTS box beside POWER FLAGS, tops aligned at
y 160.02, wired the same way. The pads are in_bom no and the footprint
is exclude_from_bom: a bare hole needs nothing bought, and the BOM
export lists no TP.

The reroute (Freerouting, 0 unrouted, 0 violations) runs /MOSI round
C2 pad 2 on B.Cu, so that pad gets one back spoke instead of two. It
still has its own GND track and full front spokes. A one-pad .kicad_dru
rule (min_resolved_spokes 1) accepts that; aimed at pad 1 instead, the
error comes back. Rejected a DRC exclusion: the key format did not match
in three tries, and the next reroute would invalidate it anyway.

The reroute also dropped 2.4's three GND vias. Measured with island
removal off and on: the back pour now loses no island, so
stitch_islands.py was not rerun.

DRC 0 errors / 3 known U2 USB-C silk warnings / 0 unconnected / 0 parity.
ERC 0. New zip 2.5_run1; 2.4_run1 stays as uploaded for Scott'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
Parts:
- added TP1: 3V3, _TestPoints:TestPoint_THTPad_D2.0mm_Drill1.0mm_P2.54, symbol Connector:TestPoint
- added TP2: GND, _TestPoints:TestPoint_THTPad_D2.0mm_Drill1.0mm_P2.54, symbol Connector:TestPoint
- added TP3: 5V, _TestPoints:TestPoint_THTPad_D2.0mm_Drill1.0mm_P2.54, symbol Connector:TestPoint
Connections:
- net +5V: now also TP3.1
- net 3V3: now also TP1.1
- net GND: now also TP2.1
Other:
- note added: "TEST POINTS TP1-TP3: probe pads"
